File: picoprobe-pcb.kicad_pcb (KiCad board)
At the start: 2 copper layers, 25 x 65.2 mm, 3 parts, among them J1 Conn_01x07_Male, J2 Conn_ARM_JTAG_SWD_10, U1 Pico

Commit message: Update to kicad 6
Connections:
- net ~TRST renamed ~{TRST}
Other:
- net class Default removed
- board text added: "~{RESET}"
- board text removed: "~RESET"

Commit message: Clean up schematic
Parts:
- J1: value Conn_01x07_Male -> Header
- J2: value Conn_ARM_JTAG_SWD_10 -> ARM
Connections:
- net SWDCLK renamed /SWDCLK
- net SWDIO renamed /SWDIO
- net SWO renamed /SWO
- net VTREF renamed /VTREF
- net ~{TRST} renamed /~{TRST}
- J1 pad 7: Net-(J1-Pad7) -> unconnected-(J1-Pin_7-Pad7)
- J2 pad 7: Net-(J2-Pad7) -> unconnected-(J2-KEY-Pad7)
- J2 pad 8: Net-(J2-Pad8) -> unconnected-(J2-NC/TDI-Pad8)
- J2 pad 9: Net-(J2-Pad9) -> unconnected-(J2-GNDDetect-Pad9)
- U1 pad 1: Net-(U1-Pad1) -> unconnected-(U1-GPIO0-Pad1)
- U1 pad 10: Net-(U1-Pad10) -> unconnected-(U1-GPIO7-Pad10)
- U1 pad 11: Net-(U1-Pad11) -> unconnected-(U1-GPIO8-Pad11)
- U1 pad 12: Net-(U1-Pad12) -> unconnected-(U1-GPIO9-Pad12)
- U1 pad 13: Net-(U1-Pad13) -> unconnected-(U1-GND-Pad13)
- U1 pad 14: Net-(U1-Pad14) -> unconnected-(U1-GPIO10-Pad14)
- U1 pad 15: Net-(U1-Pad15) -> unconnected-(U1-GPIO11-Pad15)
- U1 pad 16: Net-(U1-Pad16) -> unconnected-(U1-GPIO12-Pad16)
- U1 pad 17: Net-(U1-Pad17) -> unconnected-(U1-GPIO13-Pad17)
- U1 pad 18: Net-(U1-Pad18) -> unconnected-(U1-GND-Pad18)
- U1 pad 19: Net-(U1-Pad19) -> unconnected-(U1-GPIO14-Pad19)
- U1 pad 2: Net-(U1-Pad2) -> unconnected-(U1-GPIO1-Pad2)
- U1 pad 20: Net-(U1-Pad20) -> unconnected-(U1-GPIO15-Pad20)
- U1 pad 21: Net-(U1-Pad21) -> unconnected-(U1-GPIO16-Pad21)
- U1 pad 22: Net-(U1-Pad22) -> unconnected-(U1-GPIO17-Pad22)
- U1 pad 23: Net-(U1-Pad23) -> unconnected-(U1-GND-Pad23)
- U1 pad 24: Net-(U1-Pad24) -> unconnected-(U1-GPIO18-Pad24)
- U1 pad 25: Net-(U1-Pad25) -> unconnected-(U1-GPIO19-Pad25)
- U1 pad 26: Net-(U1-Pad26) -> unconnected-(U1-GPIO20-Pad26)
- U1 pad 27: Net-(U1-Pad27) -> unconnected-(U1-GPIO21-Pad27)
- U1 pad 28: Net-(U1-Pad28) -> unconnected-(U1-GND-Pad28)
- U1 pad 29: Net-(U1-Pad29) -> unconnected-(U1-GPIO22-Pad29)
- U1 pad 3: Net-(U1-Pad3) -> unconnected-(U1-GND-Pad3)
- U1 pad 30: Net-(U1-Pad30) -> unconnected-(U1-RUN-Pad30)
- U1 pad 31: Net-(U1-Pad31) -> unconnected-(U1-GPIO26_ADC0-Pad31)
- U1 pad 32: Net-(U1-Pad32) -> unconnected-(U1-GPIO27_ADC1-Pad32)
- U1 pad 33: Net-(U1-Pad33) -> unconnected-(U1-AGND-Pad33)
- U1 pad 35: Net-(U1-Pad35) -> unconnected-(U1-ADC_VREF-Pad35)
- U1 pad 36: Net-(U1-Pad36) -> unconnected-(U1-3V3-Pad36)
- U1 pad 37: Net-(U1-Pad37) -> unconnected-(U1-3V3_EN-Pad37)
- U1 pad 38: Net-(U1-Pad38) -> unconnected-(U1-GND-Pad38)
- U1 pad 39: Net-(U1-Pad39) -> unconnected-(U1-VSYS-Pad39)
- U1 pad 40: Net-(U1-Pad40) -> unconnected-(U1-VBUS-Pad40)
- U1 pad 41: Net-(U1-Pad41) -> unconnected-(U1-SWCLK-Pad41)
- U1 pad 42: Net-(U1-Pad42) -> unconnected-(U1-GND-Pad42)
- U1 pad 43: Net-(U1-Pad43) -> unconnected-(U1-SWDIO-Pad43)
- U1 pad 9: Net-(U1-Pad9) -> unconnected-(U1-GPIO6-Pad9)
